Commit message: Fix movement with arm
Robot can be driven with the arm attach

File: moveo_urdf/urdf/moveo_urdf.urdf (robot description, URDF)
Before this commit: robot turtlebot3_waffle_pi, 22 links, 21 joints
Joints:
- joint Joint_1: origin xyz=0 0 0.1 rpy=0 0 0 -> xyz=0 0 0.3 rpy=0 0 0

File: robutler_description/urdf/robutler.urdf.xacro (robot description, xacro)
@@ -26,5 +26,5 @@
     <inertial>
       <origin xyz="0 0 0" rpy="0 0 0"/>
-      <mass value="1.3729096e+00"/>
+      <mass value="1.3729096e+01"/>
       <inertia ixx="8.7002718e-03" ixy="-4.7576583e-05" ixz="1.1160499e-04"
                iyy="8.6195418e-03" iyz="-3.5422299e-06"
@@ -263,5 +263,5 @@
         </collision>
 	<inertial>
-            <mass value="0.1" />
+            <mass value="0.01" />
             <inertia ixx="0.03" iyy="0.03" izz="0.03" ixy="0.0" ixz="0.0" iyz="0.0" />
         </inertial>
@@ -284,5 +284,5 @@
         </collision>
 	<inertial>
-            <mass value="0.1" />
+            <mass value="0.01" />
             <inertia ixx="0.03" iyy="0.03" izz="0.03" ixy="0.0" ixz="0.0" iyz="0.0" />
         </inertial>
@@ -312,5 +312,5 @@
         </collision>
 	<inertial>
-            <mass value="0.1" />
+            <mass value="0.01" />
             <inertia ixx="0.03" iyy="0.03" izz="0.03" ixy="0.0" ixz="0.0" iyz="0.0" />
         </inertial>
@@ -340,5 +340,5 @@
         </collision>
 	<inertial>
-            <mass value="0.1" />
+            <mass value="0.01" />
             <inertia ixx="0.03" iyy="0.03" izz="0.03" ixy="0.0" ixz="0.0" iyz="0.0" />
         </inertial>
@@ -368,5 +368,5 @@
         </collision>
 	<inertial>
-            <mass value="0.1" />
+            <mass value="0.01" />
             <inertia ixx="0.03" iyy="0.03" izz="0.03" ixy="0.0" ixz="0.0" iyz="0.0" />
         </inertial>
@@ -396,5 +396,5 @@
         </collision>
 	<inertial>
-            <mass value="0.1" />
+            <mass value="0.01" />
             <inertia ixx="0.03" iyy="0.03" izz="0.03" ixy="0.0" ixz="0.0" iyz="0.0" />
         </inertial>
@@ -424,5 +424,5 @@
         </collision>
 				<inertial>
-            <mass value="0.1" />
+            <mass value="0.01" />
             <inertia ixx="0.03" iyy="0.03" izz="0.03" ixy="0.0" ixz="0.0" iyz="0.0" />
         </inertial>
@@ -452,5 +452,5 @@
         </collision>
 				<inertial>
-            <mass value="0.1" />
+            <mass value="0.01" />
             <inertia ixx="0.03" iyy="0.03" izz="0.03" ixy="0.0" ixz="0.0" iyz="0.0" />
         </inertial>
@@ -473,5 +473,5 @@
         </collision>
 				<inertial>
-            <mass value="0.1" />
+            <mass value="0.01" />
             <inertia ixx="0.03" iyy="0.03" izz="0.03" ixy="0.0" ixz="0.0" iyz="0.0" />
         </inertial>
@@ -510,5 +510,5 @@
         </collision>
 				<inertial>
-            <mass value="0.1" />
+            <mass value="0.01" />
             <inertia ixx="0.03" iyy="0.03" izz="0.03" ixy="0.0" ixz="0.0" iyz="0.0" />
         </inertial>
@@ -539,5 +539,5 @@
         </collision>
 				<inertial>
-            <mass value="0.1" />
+            <mass value="0.01" />
             <inertia ixx="0.03" iyy="0.03" izz="0.03" ixy="0.0" ixz="0.0" iyz="0.0" />
         </inertial>

Commit message: Fix joint gripper limits

File: moveo_urdf/urdf/moveo_urdf.urdf (robot description, URDF)
Before this commit: robot turtlebot3_waffle_pi, 22 links, 21 joints
Joints:
- joint Tip_Gripper_Idol_Joint: limit lower=3.14 upper=-3.14 effort=100 velocity=0.5 -> lower=-3.14 upper=3.14 effort=100 velocity=0.5
