Commit message: fix joint limit in another urdf

File: robutler_description/urdf/robutler.urdf.xacro (robot description, xacro)
@@ -490,5 +490,5 @@
         <child link="Tip_Gripper_Idol" />
         <axis xyz="0 1 0" />
-        <limit lower="3.14" upper="-3.14" effort="100" velocity="0.5" />
+        <limit lower="-3.14" upper="3.14" effort="100" velocity="0.5" />
         <mimic joint="Gripper_Idol_Gear_Joint" multiplier="-1" offset="0" />
     </joint>

Commit message: Adding the new camera geometry and the base

File: robutler_description/urdf/robutler.urdf.xacro (robot description, xacro)
@@ -562,5 +562,5 @@
       <origin xyz="0.005 0.011 0.013" rpy="0 0 0"/>
       <geometry>
-        <box size="1 1 1"/>
+        <box size="0 0 0"/>
       </geometry>
     </collision>

Commit message: Add  pose to the moveit configuration, urdf changes, alter camera topic
Add a traveling pose to the moveit configuration. 
Add geometry to the camera in the robot arm, delete the  geometry from the origiunal camera. Add more mass to the robot base top improve stability. Alter the cameara topic for the camera node

File: robutler_description/urdf/robutler.urdf.xacro (robot description, xacro)
@@ -171,5 +171,5 @@
       <origin xyz="0.005 0.011 0.013" rpy="0 0 0"/>
       <geometry>
-        <box size="0.015 0.030 0.027"/>
+        <box size="0.0 0.0 0.0"/>
       </geometry>
     </collision>
@@ -203,5 +203,5 @@
     </collision>
     <inertial>
-      <mass value="0.01"/>
+      <mass value="1.0"/>
       <origin xyz="0 0 0" rpy="0 0 0"/>
       <inertia ixx="0.01" ixy="0.0" ixz="0.01" iyy="0.0" iyz="0.0" izz="0.0"/>
@@ -562,5 +562,5 @@
       <origin xyz="0.005 0.011 0.013" rpy="0 0 0"/>
       <geometry>
-        <box size="0 0 0"/>
+        <box size="0.015 0.030 0.027"/>
       </geometry>
     </collision>
