Commit message: Changes to the moveit launch file, gazebo config, and urdf
Adding a second camera to the robot, remove the spawn of the robot when launching moveit, and adding the support base for the arm. Also changing the wheel values to support the new weigh

File: robutler_description/urdf/robutler.gazebo.xacro (robot description, xacro)
@@ -71,6 +71,6 @@
       <wheelSeparation>0.287</wheelSeparation>
       <wheelDiameter>0.066</wheelDiameter>
-      <wheelAcceleration>1</wheelAcceleration>
-      <wheelTorque>10</wheelTorque>
+      <wheelAcceleration>10</wheelAcceleration>
+      <wheelTorque>10000000000</wheelTorque>
       <rosDebugLevel>na</rosDebugLevel>
     </plugin>
@@ -176,4 +176,43 @@
     </plugin>
   </gazebo>
+  <gazebo reference="camera_rgb_frame_arm">
+    <sensor type="camera" name="Pi Camera">
+      <always_on>true</always_on>
+      <visualize>$(arg camera_visual)</visualize>
+      <camera>
+          <horizontal_fov>1.085595</horizontal_fov>
+          <image>
+              <width>640</width>
+              <height>480</height>
+              <format>R8G8B8</format>
+          </image>
+          <clip>
+              <near>0.03</near>
+              <far>100</far>
+          </clip>
+      </camera>
+      <plugin name="camera_controller" filename="libgazebo_ros_camera.so">
+        <alwaysOn>true</alwaysOn>
+        <updateRate>30.0</updateRate>
+        <cameraName>camera</cameraName>
+        <frameName>camera_rgb_optical_frame</frameName>
+        <imageTopicName>rgb/image_raw_arm</imageTopicName>
+        <cameraInfoTopicName>rgb/camera_info_arm</cameraInfoTopicName>
+        <hackBaseline>0.07</hackBaseline>
+        <distortionK1>0.0</distortionK1>
+        <distortionK2>0.0</distortionK2>
+        <distortionK3>0.0</distortionK3>
+        <distortionT1>0.0</distortionT1>
+        <distortionT2>0.0</distortionT2>
+      </plugin>
+    </sensor>
+  </gazebo>
+  <gazebo>
+    <plugin filename="libgazebo_ros_control.so" name="gazebo_ros_control">
+      <robotNamespace>/moveo_urdf</robotNamespace>
+      <robotSimType>gazebo_ros_control/DefaultRobotHWSim</robotSimType>
+      <legacyModeNS>true</legacyModeNS>
+    </plugin>
+  </gazebo>
     <transmission name="trans1">
       <type>transmission_interface/SimpleTransmission</type>

File: robutler_description/urdf/robutler.urdf.xacro (robot description, xacro)
@@ -187,9 +187,9 @@
   </joint>
   <link name="camera_rgb_optical_frame"/>
-<!-- ...................................................Robot TO MANIPULATOR ................................
+<!-- ...................................................Robot TO MANIPULATOR ................................ -->
   <link name="base_for_arm">
     <visual>
       <geometry>
-        <cylinder radius="0.15" length="0.04"/>
+        <cylinder radius="0.1" length="0.04"/>
       </geometry>
       <material name="black">
@@ -199,5 +199,5 @@
     <collision>
       <geometry>
-        <cylinder radius="0.15" length="0.04"/>
+        <cylinder radius="0.1" length="0.04"/>
       </geometry>
     </collision>
@@ -205,5 +205,5 @@
       <mass value="10.0"/>
       <origin xyz="0 0 0" rpy="0 0 0"/>
-      <inertia ixx="0.083333" ixy="0.0" ixz="0.0" iyy="0.083333" iyz="0.0" izz="0.166667"/>
+      <inertia ixx="0.043333" ixy="0.0" ixz="0.0" iyy="0.023333" iyz="0.0" izz="0.086667"/>
     </inertial>
   </link>
@@ -237,5 +237,5 @@
         <parent link="base_scan" />
         <child link="base_for_arm" />
-    </joint>-->
+    </joint>
 <!-- ...................................................MANIPULATOR ................................ -->
     <joint name="Joint_1" type="revolute">
@@ -243,5 +243,5 @@
         <axis xyz="0 0 1" />
         <limit lower="-1.5707963268" upper="1.5707963268" effort="100" velocity="1.919862177191" />
-        <parent link="base_scan" />
+        <parent link="cylinder" />
         <child link="Link_1" />
     </joint>
@@ -551,3 +551,30 @@
         <mimic joint="Gripper_Idol_Gear_Joint" multiplier="1" offset="0" />
     </joint>
+  <!-- ________________________________NEW CAMERA Configuration _________________________________________________-->
+  <joint name="camera_joint_arm" type="fixed">
+    <!-- <origin xyz="0.073 -0.011 0.084" rpy="0 0 0"/> -->
+    <origin xyz="0 0 0" rpy="0 0 0"/>
+    <parent link="Link_5"/>
+    <child link="camera_link_arm"/>
+  </joint>
+  <link name="camera_link_arm">
+    <collision>
+      <origin xyz="0.005 0.011 0.013" rpy="0 0 0"/>
+      <geometry>
+        <box size="1 1 1"/>
+      </geometry>
+    </collision>
+  </link>
+  <joint name="camera_rgb_joint_arm" type="fixed">
+    <origin xyz="0 0 0.1" rpy="0 -1.57 -1.57"/>
+    <parent link="camera_link_arm"/>
+    <child link="camera_rgb_frame_arm"/>
+  </joint>
+  <link name="camera_rgb_frame_arm"/>
+  <joint name="camera_rgb_optical_joint_arm" type="fixed">
+    <origin xyz="0 0 0" rpy="0 0 0"/>
+    <parent link="camera_rgb_frame_arm"/>
+    <child link="camera_rgb_optical_frame_arm"/>
+  </joint>
+  <link name="camera_rgb_optical_frame_arm"/>
 </robot>

Commit message: Adding the arm camera, and the support base for the arm
Camera added and aligned with the gripper, the base is working, it's necessary to adjust the weight of the turtlebot.

File: robutler_description/urdf/robutler.gazebo.xacro (robot description, xacro)
@@ -169,4 +169,44 @@
     </sensor>
   </gazebo>
+<!-- Second Camera -->
+  <gazebo reference="camera_rgb_frame_arm">
+    <sensor type="camera" name="Pi Camera">
+      <always_on>true</always_on>
+      <visualize>$(arg camera_visual)</visualize>
+      <camera>
+          <horizontal_fov>1.085595</horizontal_fov>
+          <image>
+              <width>640</width>
+              <height>480</height>
+              <format>R8G8B8</format>
+          </image>
+          <clip>
+              <near>0.03</near>
+              <far>100</far>
+          </clip>
+      </camera>
+      <plugin name="camera_controller" filename="libgazebo_ros_camera.so">
+        <alwaysOn>true</alwaysOn>
+        <updateRate>30.0</updateRate>
+        <cameraName>camera</cameraName>
+        <frameName>camera_rgb_optical_frame_arm</frameName>
+        <imageTopicName>rgb/image_raw_arm</imageTopicName>
+        <cameraInfoTopicName>rgb/camera_info_arm</cameraInfoTopicName>
+        <hackBaseline>0.07</hackBaseline>
+        <distortionK1>0.0</distortionK1>
+        <distortionK2>0.0</distortionK2>
+        <distortionK3>0.0</distortionK3>
+        <distortionT1>0.0</distortionT1>
+        <distortionT2>0.0</distortionT2>
+      </plugin>
+    </sensor>
+  </gazebo>
+  <gazebo>
+    <plugin filename="libgazebo_ros_control.so" name="gazebo_ros_control">
+      <robotNamespace>/moveo_urdf</robotNamespace>
+      <robotSimType>gazebo_ros_control/DefaultRobotHWSim</robotSimType>
+      <legacyModeNS>true</legacyModeNS>
+    </plugin>
+  </gazebo>
   <gazebo>
     <plugin filename="libgazebo_ros_control.so" name="gazebo_ros_control">

File: robutler_description/urdf/robutler.urdf.xacro (robot description, xacro)
@@ -187,9 +187,9 @@
   </joint>
   <link name="camera_rgb_optical_frame"/>
-<!-- ...................................................Robot TO MANIPULATOR ................................
+<!-- ...................................................Robot TO MANIPULATOR ................................ -->
   <link name="base_for_arm">
     <visual>
       <geometry>
-        <cylinder radius="0.15" length="0.04"/>
+        <cylinder radius="0.02" length="0.04"/>
       </geometry>
       <material name="black">
@@ -199,11 +199,11 @@
     <collision>
       <geometry>
-        <cylinder radius="0.15" length="0.04"/>
-      </geometry>
-    </collision>
-    <inertial>
-      <mass value="10.0"/>
+        <cylinder radius="0.02" length="0.04"/>
+      </geometry>
+    </collision>
+    <inertial>
+      <mass value="0.01"/>
       <origin xyz="0 0 0" rpy="0 0 0"/>
-      <inertia ixx="0.083333" ixy="0.0" ixz="0.0" iyy="0.083333" iyz="0.0" izz="0.166667"/>
+      <inertia ixx="0.01" ixy="0.0" ixz="0.01" iyy="0.0" iyz="0.0" izz="0.0"/>
     </inertial>
   </link>
@@ -223,7 +223,7 @@
     </collision>
     <inertial>
-      <mass value="2.0"/>
+      <mass value="0.01"/>
       <origin xyz="0 0 0" rpy="0 0 0"/>
-      <inertia ixx="0.002667" ixy="0.0" ixz="0.0" iyy="0.002667" iyz="0.0" izz="0.005333"/>
+      <inertia ixx="0.01" ixy="0.0" ixz="0.01" iyy="0.0" iyz="0.0" izz="0.0"/>
     </inertial>
   </link>
@@ -237,11 +237,11 @@
         <parent link="base_scan" />
         <child link="base_for_arm" />
-    </joint>-->
+    </joint>
 <!-- ...................................................MANIPULATOR ................................ -->
-    <joint name="Joint_1" type="revolute">
-	<origin xyz="0 0 0.1" rpy="0 0 0" />
+  <joint name="Joint_1" type="revolute">
+	  <origin xyz="0 0 0.1" rpy="0 0 0" />
         <axis xyz="0 0 1" />
         <limit lower="-1.5707963268" upper="1.5707963268" effort="100" velocity="1.919862177191" />
-        <parent link="base_scan" />
+        <parent link="cylinder" />
         <child link="Link_1" />
     </joint>
@@ -551,3 +551,30 @@
         <mimic joint="Gripper_Idol_Gear_Joint" multiplier="1" offset="0" />
     </joint>
+ <!-- ________________________________NEW CAMERA Configuration _________________________________________________-->
+  <joint name="camera_joint_arm" type="fixed">
+    <!-- <origin xyz="0.073 -0.011 0.084" rpy="0 0 0"/> -->
+    <origin xyz="0 0 0" rpy="0 0 0"/>
+    <parent link="Link_5"/>
+    <child link="camera_link_arm"/>
+  </joint>
+  <link name="camera_link_arm">
+    <collision>
+      <origin xyz="0.005 0.011 0.013" rpy="0 0 0"/>
+      <geometry>
+        <box size="1 1 1"/>
+      </geometry>
+    </collision>
+  </link>
+  <joint name="camera_rgb_joint_arm" type="fixed">
+    <origin xyz="0 0 0.1" rpy="0 -1.57 -1.57"/>
+    <parent link="camera_link_arm"/>
+    <child link="camera_rgb_frame_arm"/>
+  </joint>
+  <link name="camera_rgb_frame_arm"/>
+  <joint name="camera_rgb_optical_joint_arm" type="fixed">
+    <origin xyz="0 0 0" rpy="0 0 0"/>
+    <parent link="camera_rgb_frame_arm"/>
+    <child link="camera_rgb_optical_frame_arm"/>
+  </joint>
+  <link name="camera_rgb_optical_frame_arm"/>
 </robot>

Commit message: Remove camera geometry

File: robutler_description/urdf/robutler.gazebo.xacro (robot description, xacro)
@@ -169,4 +169,44 @@
     </sensor>
   </gazebo>
+<!-- Second Camera -->
+  <gazebo reference="camera_rgb_frame_arm">
+    <sensor type="camera" name="Pi Camera">
+      <always_on>true</always_on>
+      <visualize>$(arg camera_visual)</visualize>
+      <camera>
+          <horizontal_fov>1.085595</horizontal_fov>
+          <image>
+              <width>640</width>
+              <height>480</height>
+              <format>R8G8B8</format>
+          </image>
+          <clip>
+              <near>0.03</near>
+              <far>100</far>
+          </clip>
+      </camera>
+      <plugin name="camera_controller" filename="libgazebo_ros_camera.so">
+        <alwaysOn>true</alwaysOn>
+        <updateRate>30.0</updateRate>
+        <cameraName>camera</cameraName>
+        <frameName>camera_rgb_optical_frame_arm</frameName>
+        <imageTopicName>rgb/image_raw_arm</imageTopicName>
+        <cameraInfoTopicName>rgb/camera_info_arm</cameraInfoTopicName>
+        <hackBaseline>0.07</hackBaseline>
+        <distortionK1>0.0</distortionK1>
+        <distortionK2>0.0</distortionK2>
+        <distortionK3>0.0</distortionK3>
+        <distortionT1>0.0</distortionT1>
+        <distortionT2>0.0</distortionT2>
+      </plugin>
+    </sensor>
+  </gazebo>
+  <gazebo>
+    <plugin filename="libgazebo_ros_control.so" name="gazebo_ros_control">
+      <robotNamespace>/moveo_urdf</robotNamespace>
+      <robotSimType>gazebo_ros_control/DefaultRobotHWSim</robotSimType>
+      <legacyModeNS>true</legacyModeNS>
+    </plugin>
+  </gazebo>
   <gazebo>
     <plugin filename="libgazebo_ros_control.so" name="gazebo_ros_control">

File: robutler_description/urdf/robutler.urdf.xacro (robot description, xacro)
@@ -551,3 +551,29 @@
         <mimic joint="Gripper_Idol_Gear_Joint" multiplier="1" offset="0" />
     </joint>
+ <!-- ________________________________NEW CAMERA Configuration _________________________________________________-->
+  <joint name="camera_joint_arm" type="fixed">
+    <origin xyz="0 0 0" rpy="0 0 0"/>
+    <parent link="Link_5"/>
+    <child link="camera_link_arm"/>
+  </joint>
+  <link name="camera_link_arm">
+    <collision>
+      <origin xyz="0.005 0.011 0.013" rpy="0 0 0"/>
+      <geometry>
+        <box size="0 0 0"/>
+      </geometry>
+    </collision>
+  </link>
+  <joint name="camera_rgb_joint_arm" type="fixed">
+    <origin xyz="0 0 0.1" rpy="0 -1.57 -1.57"/>
+    <parent link="camera_link_arm"/>
+    <child link="camera_rgb_frame_arm"/>
+  </joint>
+  <link name="camera_rgb_frame_arm"/>
+  <joint name="camera_rgb_optical_joint_arm" type="fixed">
+    <origin xyz="0 0 0" rpy="0 0 0"/>
+    <parent link="camera_rgb_frame_arm"/>
+    <child link="camera_rgb_optical_frame_arm"/>
+  </joint>
+  <link name="camera_rgb_optical_frame_arm"/>
 </robot>

Commit message: Remove unused dir, and adding the kinect camera

File: robutler_description/urdf/robutler.gazebo.xacro (robot description, xacro)
@@ -137,8 +137,46 @@
   </gazebo>
 <!--link : https://www.raspberrypi.org/documentation/hardware/camera/-->
-  <gazebo reference="camera_rgb_frame">
-    <sensor type="camera" name="Pi Camera">
-      <always_on>true</always_on>
-      <visualize>$(arg camera_visual)</visualize>
+ <!-- <gazebo reference="camera_rgb_frame">
+   <sensor name="world" type="depth">
+        <pose frame="world">0.0 0.0 1.0 0.0 -1.5708 1.5708</pose>
+        <camera>
+            <horizontal_fov>0.74839718</horizontal_fov>
+            <image>
+                <width>1280</width>
+                <height>1024</height>
+                <format>L_INT8</format>
+            </image>
+            <clip>
+                <near>0.1</near>
+                <far>10.0</far>
+            </clip>
+            <noise>
+                <type>gaussian</type>
+                <mean>0.5</mean>
+                <stddev>1.0</stddev>
+            </noise>
+        </camera>
+        <plugin name="kinect_plugin" filename="libgazebo_ros_openni_kinect.so">
+            <baseline>0.1</baseline>
+            <alwaysOn>true</alwaysOn>
+            <updateRate>30.0</updateRate>
+            <cameraName>kinect_test</cameraName>
+            <imageTopicName>/camera/depth_registered/image_raw</imageTopicName>
+            <cameraInfoTopicName>/depth/camera_info</cameraInfoTopicName>
+            <depthImageTopicName>/depth/image_raw_depth</depthImageTopicName>
+            <depthImageInfoTopicName>/depth/camera_info</depthImageInfoTopicName>
+            <pointCloudTopicName>filtered_cloud</pointCloudTopicName>
+            <frameName>camera_rgb_optical_frame</frameName>
+            <pointCloudCutoff>0.5</pointCloudCutoff>
+            <pointCloudCutoffMax>2.0</pointCloudCutoffMax>
+        </plugin>
+        <always_on>true</always_on>
+        <update_rate>1.0</update_rate>
+    </sensor>
+  </gazebo>-->
+ <gazebo reference="camera_rgb_frame">
+    <sensor type="depth" name="kinect">
+      <always_on>1</always_on>
+      <visualize>true</visualize>
       <camera>
           <horizontal_fov>1.085595</horizontal_fov>
@@ -148,4 +186,6 @@
               <format>R8G8B8</format>
           </image>
+          <depth_camera>
+          </depth_camera>
           <clip>
               <near>0.03</near>
@@ -153,19 +193,34 @@
           </clip>
       </camera>
-      <plugin name="camera_controller" filename="libgazebo_ros_camera.so">
-        <alwaysOn>true</alwaysOn>
-        <updateRate>30.0</updateRate>
-        <cameraName>camera</cameraName>
-        <frameName>camera_rgb_optical_frame</frameName>
-        <imageTopicName>rgb/image_raw</imageTopicName>
-        <cameraInfoTopicName>rgb/camera_info</cameraInfoTopicName>
-        <hackBaseline>0.07</hackBaseline>
-        <distortionK1>0.0</distortionK1>
-        <distortionK2>0.0</distortionK2>
-        <distortionK3>0.0</distortionK3>
-        <distortionT1>0.0</distortionT1>
-        <distortionT2>0.0</distortionT2>
+      <plugin name="kinect_plugin" filename="libgazebo_ros_openni_kinect.so">
+          <alwaysOn>true</alwaysOn>
+          <updateRate>10.0</updateRate>
+          <cameraName>kinect</cameraName>
+          <imageTopicName>/camera/depth_registered/image_raw</imageTopicName>
+          <cameraInfoTopicName>/depth/camera_info</cameraInfoTopicName>
+          <depthImageTopicName>/depth/image_raw_depth</depthImageTopicName>
+          <depthImageInfoTopicName>/depth/camera_info</depthImageInfoTopicName>
+          <pointCloudTopicName>filtered_cloud</pointCloudTopicName>
+          <frameName>camera_rgb_optical_frame</frameName>
+          <pointCloudCutoff>0.01</pointCloudCutoff>
+          <hackBaseline>0.07</hackBaseline>
+          <distortionK1>0.0</distortionK1>
+          <distortionK2>0.0</distortionK2>
+          <distortionK3>0.0</distortionK3>
+          <distortionT1>0.0</distortionT1>
+          <distortionT2>0.0</distortionT2>
+          <CxPrime>0.0</CxPrime>
+          <Cx>0.0</Cx>
+          <Cy>0.0</Cy>
+          <focalLenmgth>0.0</focalLenmgth>
       </plugin>
     </sensor>
+  </gazebo>
+  <gazebo>
+    <plugin filename="libgazebo_ros_control.so" name="gazebo_ros_control">
+      <robotNamespace>/moveo_urdf</robotNamespace>
+      <robotSimType>gazebo_ros_control/DefaultRobotHWSim</robotSimType>
+      <legacyModeNS>true</legacyModeNS>
+    </plugin>
   </gazebo>
 <!-- Second Camera -->

File: robutler_description/urdf/robutler.urdf.xacro (robot description, xacro)
@@ -168,4 +168,10 @@
   </joint>
   <link name="camera_link">
+    <visual>
+      <origin xyz="0.005 0.011 0.013" rpy="0 0 0"/>
+      <geometry>
+        <box size="0.0 0.0 0.0"/>
+      </geometry>
+    </visual>
     <collision>
       <origin xyz="0.005 0.011 0.013" rpy="0 0 0"/>
